File: REF03.kicad_sch (KiCad schematic)
At the start: 20 parts, among them SW1 SW_SPST, U1 SN74LVC2G14DBV, U2 REF03GP

Commit message: Updated README
Parts:
- added C7: 10u, Capacitor_SMD:C_0805_2012Metric, symbol Device:C
- added FB1: FerriteBead, Inductor_SMD:L_0805_2012Metric, symbol Device:FerriteBead
Connections:
- net GND: now also C7.1
- net at C6.2, R3.1, U2.6 (VOUT): now also FB1.1; no longer TP1.1
- new net: C7.2, FB1.2, TP1.1
Other:
- moved on the sheet: TP1
